File: THE BLIME AIO FC.kicad_pcb (KiCad board)
At the start: 6 copper layers, 38.7 x 40.8 mm, 32 parts, among them J1 Conn_01x16_Pin, J10 Conn_01x01_Socket, J11 Conn_01x01_Socket, J12 Conn_01x01_Socket, J13 Conn_01x01_Socket, J14 Conn_01x01_Socket, J15 Conn_01x01_Socket, J2 Conn_01x01_Socket, J3 Conn_01x01_Socket, J4 Conn_01x01_Socket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

Commit message: Add files via upload
Routing:
- net GND: track 71.6 -> 142.5 mm, vias 27 -> 44
- net PHASE G: track 5.60 -> 35.0 mm, vias 2 -> 10
- net +BATT: track 15.4 -> 42.1 mm, vias 3 -> 14
- net M3-4: track 44.8 -> 47.8 mm, vias 0 -> 1
